File: Crocker-ElectricSchematic/Crocker-ElectricSchematic.kicad_sch (KiCad schematic)
At the start: 0 parts

Commit message: electrical schematic
Parts:
- added BT1: 12V Battery, symbol Device:Battery
- added D?: D, symbol Device:D
- added L1: ElectromagneticActor, symbol Device:ElectromagneticActor
- added U1: XIAO-ESP32-S3-SMD, Seeed_Studio_XIAO_Series:XIAO-ESP32-S3-SMD, symbol SEED Studio:XIAO-ESP32-S3-SMD
- added U2, U?: LM2596S-5, Package_TO_SOT_SMD:TO-263-5_TabPin3, symbol Regulator_Switching:LM2596S-5
Connections:
- new net: BT1.1 (+), D?.1 (K), L1.1 (-), U2.1 (VIN+), U?.3 (LOAD+)
- new net: D?.2 (A), L1.2 (+), U?.4 (LOAD-)
- new net 23VBAT: U2.3 (VOUT+)
- new net 24 GND: BT1.2 (-), U2.2 (VIN-), U?.2 (GND)
- new net 24GND: U2.4 (VOUT-)
- new net ESP32 PIN: U?.1 (PWM)
Other:
- company: (none) -> ChompSafe
- title: (none) -> ElectroMagnet Schematic
